File: board/biscuit.sch (KiCad schematic (older format))
At the start: 3 parts

Commit message: movement on the schematic
Parts:
- added C? (x3): CSMALL, symbol CSMALL
- added P?: CONN_3X2, symbol CONN_3X2
- added Q? (x5): FET, symbol MOSFET_P
- added Q? (x5): NPN, TO92-EBC, symbol BC237
- added R? (x11): R, symbol R
- added SW?: SW_PUSH, symbol SW_PUSH
- added U?: ATMEGA168, MODULE, symbol ATMEGA168
- added X?: CRYSTAL, symbol CRYSTAL
- U?: value 7805 -> AP1084
Connections:
- net labels added: CH1, CH2, CH3, CH4, CH5, PB1, PB2, PB3, PD5, PD6
- wire segments 4 -> 96
Other:
- moved on the sheet: C?, U?

Commit message: schematic is close to being done
Parts:
- removed C? (x2): C, symbol C
- removed C? (x3): CSMALL, symbol CSMALL
- removed P?: CONN_3X2, symbol CONN_3X2
- removed U?: ATMEGA168, MODULE, symbol ATMEGA168
- removed X?: CRYSTAL, symbol CRYSTAL
- added C? (x3): 0.1uF, symbol C
- added C? (x2): 100uF, symbol CP1
- added C? (x4): 50pF, symbol C
- added D?: 1N4004, symbol DIODE
- added IC?: ATMEGA328-P, DIL28, symbol ATMEGA328-P
- added J?: OUT, symbol RJ45
- added J?: IN, symbol RJ45
- added JP?: JUMPER, symbol JUMPER
- added P?: TTL-232R, symbol CONN_6
- added P?: ICSP, symbol CONN_3X2
- added P?: CONN_6X2, symbol CONN_6X2
- added P?: CONN_4, symbol CONN_4
- added Q?: FET, symbol MOSFET_P
- added Q?: NPN, TO92-EBC, symbol BC237
- added R? (x2): 10k, symbol R
- added R?: 100 1/2W, symbol R
- added R?: 120, symbol R
- added R? (x2): R, symbol R
- added R? (x8): 10M, symbol R
- added U?: MAX485, symbol MAX485
- added Y?: RESONATOR, symbol RESONATOR
- U?: value AP1084 -> AP1084T50L
Connections:
- net labels added: +12V, CHRG, CTRLDE, CTRLRE, LCH1, LCH2, LCH3, LCH4, LCH5, LCH6, LPN1, LPN2, LPN3, LPN4, LPN5, LPN6, MISO, MOSI, RESET, RXD, SCK, TCH1, TCH2, TCH3, TCH4, TPN1, TPN2, TPN3, TPN4, TXD, VCC
- net labels removed: +5V, CH1, CH2, CH3, CH4, CH5, PB1, PB2, PB3, PD5, PD6, VAA
- wire segments 96 -> 226
- no-connect marks 0 -> 8
Other:
- moved on the sheet: Q?, R?, SW?, U?

Commit message: v1 of board
Parts:
- removed P?: CONN_4, symbol CONN_4
- removed Q? (x6): FET, symbol MOSFET_P
- removed Q? (x6): NPN, TO92-EBC, symbol BC237
- removed R? (x12): R, symbol R
- removed SW?: SW_PUSH, symbol SW_PUSH
- added D2: BI_LED, symbol BI_LED
- added JP2: JUMPER, symbol JUMPER
- added P1: PWR_IN, symbol CONN_2
- added P2: PWR_OUT, symbol CONN_2
- added P6: CONN_4X2, symbol CONN_4X2
- added Q1, Q10, Q2, Q5, Q6, Q9: FET, symbol MOSFET_P
- added Q11, Q12, Q3, Q4, Q7, Q8: NPN, TO92-EBC, symbol BC237
- added R15, R16, R21, R22, R26, R27: 2 1/2W, symbol R
- added R17, R18, R23, R24, R5, R6: 10K, symbol R
- added R19: 150, symbol R
- added R20: 120, symbol R
- added RV1, RV2, RV3, RV4, RV5, RV6: 10 1/2W, symbol POT
- C3, C4, C5, C6: renamed from C?; value 50pF -> 100pF
- R11, R13, R7, R9: renamed from R?; value 10M -> 10K
- R25: renamed from R?; value R -> 10K
- gave numbers to parts that had none: 24
Connections:
- net labels added: GNDA, GRN, INTERFACES, LED DRIVERS, MCU, POWER, RED, RS-485, TOUCH DRIVERS
- wire segments 226 -> 246
- no-connect marks 8 -> 15
Other:
- moved on the sheet: C1, C2, C3, C4, C5, C6, C7, C8, C9, D1, IC1, J1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

Commit message: reality check
Parts:
- removed C8, C9: 100uF, symbol CP1
- removed JP2: JUMPER, symbol JUMPER
- removed P6: CONN_4X2, symbol CONN_4X2
- removed RV1, RV2, RV3, RV4, RV5: 10 1/2W, symbol POT
- added C8: .33uF, symbol C
- added C9: .1uF, symbol C
- added JP2: CONN_3, symbol CONN_3
- added P6: CONN_4, symbol CONN_4
- R10, R12, R14, R8: value 10M -> 10K
- R11, R13, R7, R9: value 10K -> 10M
- R15: value 2 1/2W -> 1.3 1W
- R16, R21, R26: value 2 1/2W -> 1.5 1W
- R22: value 2 1/2W -> .75 1W
- U2: value AP1084T50L -> 7805
Connections:
- net labels added: DGND
- no-connect marks 15 -> 13
